Commit message: Robot Model added with complete launch files. This includes the jackal_race.world map

File: urdf/udacity_bot.xacro (robot description, xacro)
@@ -1,5 +1,8 @@
 <?xml version='1.0'?>
 <robot name="udacity_bot" xmlns:xacro="http://www.ros.org/wiki/xacro">
+  <xacro:include filename="$(find udacity_bot)/urdf/udacity_bot.gazebo" />
+  <!--                             Base link                                 -->
   <link name="robot_footprint"></link>
+  <!--                              Joints                                  -->
   <joint name="robot_footprint_joint" type="fixed">
     <origin xyz="0 0 0" rpy="0 0 0" />
@@ -7,5 +10,5 @@
     <child link="chassis" />
   </joint>
-  <joint type="continuous" name="left_wheel_hinge">
+  <joint name="left_wheel_hinge" type="continuous">
     <origin xyz="0 0.15 0" rpy="0 0 0"/>
     <child link="left_wheel"/>
@@ -15,5 +18,5 @@
     <dynamics damping="1.0" friction="1.0"/>
   </joint>
-  <joint type="continuous" name="right_wheel_hinge">
+  <joint name="right_wheel_hinge" type="continuous">
     <origin xyz="0 -0.15 0" rpy="0 0 0"/>
     <child link="right_wheel"/>
@@ -23,4 +26,16 @@
     <dynamics damping="1.0" friction="1.0"/>
   </joint>
+  <!-- Sensor Joints -->
+  <joint name="camera_joint" type="fixed">
+    <origin xyz="0.2 0 0" rpy="0 0 0" />
+    <parent link="chassis"/>
+    <child link="camera" />
+  </joint>
+  <joint name="hokuyo_joint" type="fixed">
+    <origin xyz="0.15 0 0.1" rpy="0 0 0" />
+    <parent link="chassis"/>
+    <child link="hokuyo" />
+  </joint>
+  <!--                               Links                                   -->
   <link name='chassis'>
     <pose>0 0 0.1 0 0 0</pose>
@@ -117,3 +132,50 @@
     </visual>
   </link>
+  <!-- Sensor Links -->
+  <link name="camera">
+    <inertial>
+      <mass value="0.1"/>
+      <origin xyz="0 0 0" rpy="0 0 0"/>
+      <inertia
+          ixx="1e-6" ixy="0" ixz="0"
+          iyy="1e-6" iyz="0"
+          izz="1e-6"
+      />
+    </inertial>
+    <collision name='camera_collision'>
+      <origin xyz="0 0 0" rpy="0 0 0"/>
+      <geometry>
+        <box size="0.05 0.05 0.05"/>
+      </geometry>
+    </collision>
+    <visual name='camera_visual'>
+      <origin xyz="0 0 0" rpy=" 0 0 0"/>
+      <geometry>
+        <box size="0.05 0.05 0.05"/>
+      </geometry>
+    </visual>
+  </link>
+  <link name="hokuyo">
+    <inertial>
+      <mass value="0.1"/>
+      <origin xyz="0 0 0" rpy="0 0 0"/>
+      <inertia
+          ixx="1e-6" ixy="0" ixz="0"
+          iyy="1e-6" iyz="0"
+          izz="1e-6"
+      />
+    </inertial>
+    <collision name='hokuyo_collision'>
+      <origin xyz="0 0 0" rpy="0 0 0"/>
+      <geometry>
+        <box size="0.1 0.1 0.1"/>
+      </geometry>
+    </collision>
+    <visual name='hokuyo_visual'>
+      <origin xyz="0 0 0" rpy=" 0 0 0"/>
+      <geometry>
+        <mesh filename="package://udacity_bot/meshes/hokuyo.dae"/>
+      </geometry>
+    </visual>
+  </link>
 </robot>

Commit message: Uploaded original code at the AMCL parameterisation for the classroom robot

File: urdf/udacity_bot.xacro (robot description, xacro)
@@ -2,7 +2,5 @@
 <robot name="udacity_bot" xmlns:xacro="http://www.ros.org/wiki/xacro">
   <xacro:include filename="$(find udacity_bot)/urdf/udacity_bot.gazebo" />
-  <!--                             Base link                                 -->
   <link name="robot_footprint"></link>
-  <!--                              Joints                                  -->
   <joint name="robot_footprint_joint" type="fixed">
     <origin xyz="0 0 0" rpy="0 0 0" />
@@ -10,32 +8,30 @@
     <child link="chassis" />
   </joint>
-  <joint name="left_wheel_hinge" type="continuous">
-    <origin xyz="0 0.15 0" rpy="0 0 0"/>
-    <child link="left_wheel"/>
+  <joint name="right_wheel_hinge" type="continuous">
+    <origin xyz="0 -0.125 0" rpy="0 0 0"/>
     <parent link="chassis"/>
-    <axis xyz="0 1 0" rpy="0 0 0"/>
+    <child link="right_wheel"/>
+    <axis xyz ="0 1 0" rpy="0 0 0"/>
     <limit effort="10000" velocity="1000"/>
     <dynamics damping="1.0" friction="1.0"/>
   </joint>
-  <joint name="right_wheel_hinge" type="continuous">
-    <origin xyz="0 -0.15 0" rpy="0 0 0"/>
-    <child link="right_wheel"/>
+  <joint name="left_wheel_hinge" type="continuous">
+    <origin xyz="0 0.125 0" rpy="0 0 0"/>
     <parent link="chassis"/>
-    <axis xyz="0 1 0" rpy="0 0 0"/>
+    <child link="left_wheel"/>
+    <axis xyz ="0 1 0" rpy="0 0 0"/>
     <limit effort="10000" velocity="1000"/>
     <dynamics damping="1.0" friction="1.0"/>
   </joint>
-  <!-- Sensor Joints -->
   <joint name="camera_joint" type="fixed">
-    <origin xyz="0.2 0 0" rpy="0 0 0" />
+    <origin xyz="0.2 0 0" rpy="0 0 0"/>
     <parent link="chassis"/>
-    <child link="camera" />
+    <child link="camera"/>
   </joint>
   <joint name="hokuyo_joint" type="fixed">
-    <origin xyz="0.15 0 0.1" rpy="0 0 0" />
+    <origin xyz="0.15 0 0.1" rpy="0 0 0"/>
     <parent link="chassis"/>
-    <child link="hokuyo" />
+    <child link="hokuyo"/>
   </joint>
-  <!--                               Links                                   -->
   <link name='chassis'>
     <pose>0 0 0.1 0 0 0</pose>
@@ -47,5 +43,5 @@
           iyy="0.1" iyz="0"
           izz="0.1"
-      />
+          />
     </inertial>
     <collision name='collision'>
@@ -86,45 +82,22 @@
     </visual>
   </link>
-  <link name="left_wheel">
+  <link name="right_wheel">
     <inertial>
       <mass value="5.0"/>
-      <origin xyz="0.0 0 0" rpy=" 0 1.5707 1.5707"/>
+      <origin xyz="0 0 0" rpy=" 0 1.5707 1.5707"/>
       <inertia
-          ixx="0.1" ixy="0" ixz="0"
-          iyy="0.1" iyz="0"
-          izz="0.1"
-      />
+            ixx="0.1" ixy="0" ixz="0"
+            iyy="0.1" iyz="0"
+            izz="0.1"
+            />
     </inertial>
-    <collision name='collision'>
-      <origin xyz="0.0 0 0" rpy=" 0 1.5707 1.5707"/>
+    <collision name="right_wheel_collision">
+      <origin xyz="0 0 0" rpy=" 0 1.5707 1.5707"/>
       <geometry>
         <cylinder radius="0.1" length="0.05"/>
       </geometry>
     </collision>
-    <visual name='chassis_visual'>
-      <origin xyz="0.0 0 0" rpy=" 0 1.5707 1.5707"/>
-      <geometry>
-        <cylinder radius="0.1" length = "0.05"/>
-      </geometry>
-    </visual>
-  </link>
-  <link name="right_wheel">
-    <inertial>
-      <mass value="5.0"/>
-      <origin xyz="0.0 0 0" rpy=" 0 1.5707 1.5707"/>
-      <inertia
-          ixx="0.1" ixy="0" ixz="0"
-          iyy="0.1" iyz="0"
-          izz="0.1"
-      />
-    </inertial>
-    <collision name='collision'>
-      <origin xyz="0.0 0 0" rpy=" 0 1.5707 1.5707"/>
-      <geometry>
-        <cylinder radius="0.1" length = "0.05"/>
-      </geometry>
-    </collision>
-    <visual name='chassis_visual'>
-      <origin xyz="0.0 0 0" rpy=" 0 1.5707 1.5707"/>
+    <visual name="right_wheel_visual">
+      <origin xyz="0 0 0" rpy=" 0 1.5707 1.5707"/>
       <geometry>
         <cylinder radius="0.1" length="0.05"/>
@@ -132,22 +105,44 @@
     </visual>
   </link>
-  <!-- Sensor Links -->
+  <link name="left_wheel">
+    <inertial>
+      <mass value="5.0"/>
+      <origin xyz="0 0 0" rpy=" 0 1.5707 1.5707"/>
+      <inertia
+          ixx="0.1" ixy="0" ixz="0"
+          iyy="0.1" iyz="0"
+          izz="0.1"
+          />
+    </inertial>
+    <collision name="left_wheel_collision">
+      <origin xyz="0 0 0" rpy=" 0 1.5707 1.5707"/>
+      <geometry>
+        <cylinder radius="0.1" length="0.05"/>
+      </geometry>
+    </collision>
+    <visual name="left_wheel_visual">
+      <origin xyz="0 0 0" rpy=" 0 1.5707 1.5707"/>
+      <geometry>
+        <cylinder radius="0.1" length="0.05"/>
+      </geometry>
+    </visual>
+  </link>
   <link name="camera">
     <inertial>
       <mass value="0.1"/>
-      <origin xyz="0 0 0" rpy="0 0 0"/>
+      <origin xyz="0 0 0" rpy=" 0 0 0"/>
       <inertia
-          ixx="1e-6" ixy="0" ixz="0"
-          iyy="1e-6" iyz="0"
-          izz="1e-6"
-      />
+        ixx="1e-6" ixy="0" ixz="0"
+        iyy="1e-6" iyz="0"
+        izz="1e-6"
+        />
     </inertial>
-    <collision name='camera_collision'>
-      <origin xyz="0 0 0" rpy="0 0 0"/>
+    <collision name="camera_collision">
+      <origin xyz="0 0 0" rpy=" 0 0 0"/>
       <geometry>
         <box size="0.05 0.05 0.05"/>
       </geometry>
     </collision>
-    <visual name='camera_visual'>
+    <visual name="camera_visual">
       <origin xyz="0 0 0" rpy=" 0 0 0"/>
       <geometry>
@@ -159,23 +154,23 @@
     <inertial>
       <mass value="0.1"/>
-      <origin xyz="0 0 0" rpy="0 0 0"/>
+      <origin xyz="0 0 0" rpy=" 0 0 0"/>
       <inertia
           ixx="1e-6" ixy="0" ixz="0"
           iyy="1e-6" iyz="0"
           izz="1e-6"
-      />
-    </inertial>
-    <collision name='hokuyo_collision'>
-      <origin xyz="0 0 0" rpy="0 0 0"/>
-      <geometry>
-        <box size="0.1 0.1 0.1"/>
-      </geometry>
-    </collision>
-    <visual name='hokuyo_visual'>
-      <origin xyz="0 0 0" rpy=" 0 0 0"/>
-      <geometry>
-        <mesh filename="package://udacity_bot/meshes/hokuyo.dae"/>
-      </geometry>
-    </visual>
-  </link>
+          />
+      </inertial>
+        <collision name="hokuyo_collision">
+            <origin xyz="0 0 0" rpy=" 0 0 0"/>
+            <geometry>
+                <box size="0.1 0.1 0.1"/>
+            </geometry>
+        </collision>
+        <visual name="hokuyo_visual">
+            <origin xyz="0 0 0" rpy=" 0 0 0"/>
+            <geometry>
+                <mesh filename="package://udacity_bot/meshes/hokuyo.dae"/>
+            </geometry>
+        </visual>
+    </link>
 </robot>
