Commit message: Final working code; Report to add

File: urdf/my_robot.xacro (robot description, xacro)
@@ -1,5 +1,14 @@
 <?xml version='1.0'?>
 <robot name="udacity_bot" xmlns:xacro="http://www.ros.org/wiki/xacro">
-  <xacro:include filename="$(find udacity_bot)/urdf/udacity_bot.gazebo" />
+  <xacro:include filename="$(find udacity_bot)/urdf/my_robot.gazebo" />
+  <material name="red">
+    <color rgba="1.0 0.0 0.0 1.0" />
+  </material>
+  <material name="green">
+    <color rgba="0.0 1.0 0.0 1.0" />
+  </material>
+  <material name="blue">
+    <color rgba="0.0 0.0 1.0 1.0" />
+  </material>
   <link name="robot_footprint"></link>
   <joint name="robot_footprint_joint" type="fixed">
@@ -9,5 +18,5 @@
   </joint>
   <joint name="right_wheel_hinge" type="continuous">
-    <origin xyz="0 -0.25 0" rpy="0 0 0"/>
+    <origin xyz="0 -0.2 0" rpy="0 0 0"/>
     <parent link="chassis"/>
     <child link="right_wheel"/>
@@ -17,5 +26,5 @@
   </joint>
   <joint name="left_wheel_hinge" type="continuous">
-    <origin xyz="0 0.25 0" rpy="0 0 0"/>
+    <origin xyz="0 0.2 0" rpy="0 0 0"/>
     <parent link="chassis"/>
     <child link="left_wheel"/>
@@ -25,10 +34,10 @@
   </joint>
   <joint name="camera_joint" type="fixed">
-    <origin xyz="0.25 0 0" rpy="0 0 0"/>
+    <origin xyz="0.2 0 0" rpy="0 0 0"/>
     <parent link="chassis"/>
     <child link="camera"/>
   </joint>
   <joint name="stem_joint" type="fixed">
-    <origin xyz="0 0 0.1" rpy="0 0 0"/>
+    <origin xyz="0.15 0 0.1" rpy="0 0 0"/>
     <parent link="chassis"/>
     <child link="stem"/>
@@ -42,5 +51,5 @@
     <pose>0 0 0.1 0 0 0</pose>
     <inertial>
-      <mass value="15.0"/>
+      <mass value="10.0"/>
       <origin xyz="0.0 0 0" rpy=" 0 0 0"/>
       <inertia
@@ -53,5 +62,5 @@
       <origin xyz="0 0 0" rpy=" 0 0 0"/>
       <geometry>
-        <cylinder radius="0.25" length="0.1"/>
+        <cylinder radius="0.2" length="0.1"/>
       </geometry>
     </collision>
@@ -59,9 +68,9 @@
       <origin xyz="0 0 0" rpy=" 0 0 0"/>
       <geometry>
-        <cylinder radius="0.25" length="0.1"/>
+        <cylinder radius="0.2" length="0.1"/>
       </geometry>
     </visual>
     <collision name='back_caster_collision'>
-      <origin xyz="-0.15 0 -0.05" rpy=" 0 0 0"/>
+      <origin xyz="-0.1 0 -0.05" rpy=" 0 0 0"/>
       <geometry>
         <sphere radius="0.0499"/>
@@ -69,5 +78,5 @@
     </collision>
     <visual name='back_caster_visual'>
-      <origin xyz="-0.15 0 -0.05" rpy=" 0 0 0"/>
+      <origin xyz="-0.1 0 -0.05" rpy=" 0 0 0"/>
       <geometry>
         <sphere radius="0.05"/>
@@ -75,5 +84,5 @@
     </visual>
     <collision name='front_caster_collision'>
-      <origin xyz="0.15 0 -0.05" rpy=" 0 0 0"/>
+      <origin xyz="0.1 0 -0.05" rpy=" 0 0 0"/>
       <geometry>
         <sphere radius="0.0499"/>
@@ -81,5 +90,5 @@
     </collision>
     <visual name='front_caster_visual'>
-      <origin xyz="0.15 0 -0.05" rpy=" 0 0 0"/>
+      <origin xyz="0.1 0 -0.05" rpy=" 0 0 0"/>
       <geometry>
         <sphere radius="0.05"/>
@@ -146,5 +155,5 @@
       <origin xyz="0 0 0" rpy="0 0 0"/>
       <geometry>
-        <box size="0.05 0.05 0.25"/>
+        <box size="0.05 0.05 0.15"/>
       </geometry>
     </collision>

File: urdf/udacity_bot.xacro (robot description, xacro)
@@ -2,4 +2,13 @@
 <robot name="udacity_bot" xmlns:xacro="http://www.ros.org/wiki/xacro">
   <xacro:include filename="$(find udacity_bot)/urdf/udacity_bot.gazebo" />
+  <material name="red">
+    <color rgba="1.0 0.0 0.0 1.0" />
+  </material>
+  <material name="green">
+    <color rgba="0.0 1.0 0.0 1.0" />
+  </material>
+  <material name="blue">
+    <color rgba="0.0 0.0 1.0 1.0" />
+  </material>
   <link name="robot_footprint"></link>
   <joint name="robot_footprint_joint" type="fixed">
@@ -7,30 +16,4 @@
     <parent link="robot_footprint"/>
     <child link="chassis" />
-  </joint>
-  <joint name="right_wheel_hinge" type="continuous">
-    <origin xyz="0 -0.125 0" rpy="0 0 0"/>
-    <parent link="chassis"/>
-    <child link="right_wheel"/>
-    <axis xyz ="0 1 0" rpy="0 0 0"/>
-    <limit effort="10000" velocity="1000"/>
-    <dynamics damping="1.0" friction="1.0"/>
-  </joint>
-  <joint name="left_wheel_hinge" type="continuous">
-    <origin xyz="0 0.125 0" rpy="0 0 0"/>
-    <parent link="chassis"/>
-    <child link="left_wheel"/>
-    <axis xyz ="0 1 0" rpy="0 0 0"/>
-    <limit effort="10000" velocity="1000"/>
-    <dynamics damping="1.0" friction="1.0"/>
-  </joint>
-  <joint name="camera_joint" type="fixed">
-    <origin xyz="0.2 0 0" rpy="0 0 0"/>
-    <parent link="chassis"/>
-    <child link="camera"/>
-  </joint>
-  <joint name="hokuyo_joint" type="fixed">
-    <origin xyz="0.15 0 0.1" rpy="0 0 0"/>
-    <parent link="chassis"/>
-    <child link="hokuyo"/>
   </joint>
   <link name='chassis'>
@@ -43,5 +26,5 @@
           iyy="0.1" iyz="0"
           izz="0.1"
-          />
+      />
     </inertial>
     <collision name='collision'>
@@ -56,4 +39,5 @@
         <box size=".4 .2 .1"/>
       </geometry>
+      <material name="blue" />
     </visual>
     <collision name='back_caster_collision'>
@@ -82,95 +66,132 @@
     </visual>
   </link>
-  <link name="right_wheel">
+  <!-- LEFT WHEEL -->
+  <joint type="continuous" name="left_wheel_hinge">
+    <origin xyz="0 0.15 0" rpy="0 0 0"/>
+    <child link="left_wheel"/>
+    <parent link="chassis"/>
+    <axis xyz="0 1 0" rpy="0 0 0"/>
+    <limit effort="10000" velocity="1000"/>
+    <dynamics damping="1.0" friction="1.0"/>
+  </joint>
+  <link name='left_wheel'>
+    <pose>0 0 0 0 1.5707 1.5707</pose>
     <inertial>
       <mass value="5.0"/>
-      <origin xyz="0 0 0" rpy=" 0 1.5707 1.5707"/>
-      <inertia
-            ixx="0.1" ixy="0" ixz="0"
-            iyy="0.1" iyz="0"
-            izz="0.1"
-            />
-    </inertial>
-    <collision name="right_wheel_collision">
-      <origin xyz="0 0 0" rpy=" 0 1.5707 1.5707"/>
-      <geometry>
-        <cylinder radius="0.1" length="0.05"/>
-      </geometry>
-    </collision>
-    <visual name="right_wheel_visual">
-      <origin xyz="0 0 0" rpy=" 0 1.5707 1.5707"/>
-      <geometry>
-        <cylinder radius="0.1" length="0.05"/>
-      </geometry>
-    </visual>
-  </link>
-  <link name="left_wheel">
-    <inertial>
-      <mass value="5.0"/>
-      <origin xyz="0 0 0" rpy=" 0 1.5707 1.5707"/>
+      <origin xyz="0 0 0" rpy="0 1.5707 1.5707" />
       <inertia
           ixx="0.1" ixy="0" ixz="0"
           iyy="0.1" iyz="0"
           izz="0.1"
-          />
+      />
     </inertial>
-    <collision name="left_wheel_collision">
-      <origin xyz="0 0 0" rpy=" 0 1.5707 1.5707"/>
+    <collision>
+      <origin xyz="0 0 0" rpy="0 1.5707 1.5707" />
       <geometry>
-        <cylinder radius="0.1" length="0.05"/>
+        <cylinder radius="0.1" length="0.05" />
       </geometry>
     </collision>
-    <visual name="left_wheel_visual">
-      <origin xyz="0 0 0" rpy=" 0 1.5707 1.5707"/>
+    <visual>
+      <origin xyz="0 0 0" rpy="0 1.5707 1.5707" />
       <geometry>
-        <cylinder radius="0.1" length="0.05"/>
+        <cylinder radius="0.1" length="0.05" />
       </geometry>
+      <material name="green" />
     </visual>
   </link>
-  <link name="camera">
+  <!-- RIGHT WHEEL -->
+  <joint type="continuous" name="right_wheel_hinge">
+    <origin xyz="0 -0.15 0" rpy="0 0 0"/>
+    <child link="right_wheel"/>
+    <parent link="chassis"/>
+    <axis xyz="0 1 0" rpy="0 0 0"/>
+    <limit effort="10000" velocity="1000"/>
+    <dynamics damping="1.0" friction="1.0"/>
+  </joint>
+  <link name='right_wheel'>
+    <pose>0 0 0 0 1.5707 1.5707</pose>
+    <inertial>
+      <mass value="5.0"/>
+      <origin xyz="0 0 0" rpy="0 1.5707 1.5707" />
+      <inertia
+          ixx="0.1" ixy="0" ixz="0"
+          iyy="0.1" iyz="0"
+          izz="0.1"
+      />
+    </inertial>
+    <collision>
+      <origin xyz="0 0 0" rpy="0 1.5707 1.5707" />
+      <geometry>
+        <cylinder radius="0.1" length="0.05" />
+      </geometry>
+    </collision>
+    <visual>
+      <origin xyz="0 0 0" rpy="0 1.5707 1.5707" />
+      <geometry>
+        <cylinder radius="0.1" length="0.05" />
+      </geometry>
+      <material name="green" />
+    </visual>
+  </link>
+  <!-- CAMERA -->
+  <joint name="camera_joint" type="fixed">
+    <origin xyz="0.2 0 0" rpy="0 0 0" />
+    <parent link="chassis" />
+    <child link="camera" />
+  </joint>
+  <link name='camera'>
+    <pose>0 0 0 0 0 0</pose>
     <inertial>
       <mass value="0.1"/>
-      <origin xyz="0 0 0" rpy=" 0 0 0"/>
-      <inertia
-        ixx="1e-6" ixy="0" ixz="0"
-        iyy="1e-6" iyz="0"
-        izz="1e-6"
-        />
-    </inertial>
-    <collision name="camera_collision">
-      <origin xyz="0 0 0" rpy=" 0 0 0"/>
-      <geometry>
-        <box size="0.05 0.05 0.05"/>
-      </geometry>
-    </collision>
-    <visual name="camera_visual">
-      <origin xyz="0 0 0" rpy=" 0 0 0"/>
-      <geometry>
-        <box size="0.05 0.05 0.05"/>
-      </geometry>
-    </visual>
-  </link>
-  <link name="hokuyo">
-    <inertial>
-      <mass value="0.1"/>
-      <origin xyz="0 0 0" rpy=" 0 0 0"/>
+      <origin xyz="0 0 0" rpy="0 0 0" />
       <inertia
           ixx="1e-6" ixy="0" ixz="0"
           iyy="1e-6" iyz="0"
           izz="1e-6"
-          />
-      </inertial>
-        <collision name="hokuyo_collision">
-            <origin xyz="0 0 0" rpy=" 0 0 0"/>
-            <geometry>
-                <box size="0.1 0.1 0.1"/>
-            </geometry>
-        </collision>
-        <visual name="hokuyo_visual">
-            <origin xyz="0 0 0" rpy=" 0 0 0"/>
-            <geometry>
-                <mesh filename="package://udacity_bot/meshes/hokuyo.dae"/>
-            </geometry>
-        </visual>
-    </link>
+      />
+    </inertial>
+    <collision>
+      <origin xyz="0 0 0" rpy=" 0 0 0" />
+      <geometry>
+        <box size="0.05 0.05 0.05" />
+      </geometry>
+    </collision>
+    <visual>
+      <origin xyz="0 0 0" rpy=" 0 0 0" />
+      <geometry>
+        <box size="0.05 0.05 0.05" />
+      </geometry>
+      <material name="red" />
+    </visual>
+  </link>
+  <!-- LASER RANGEFINDER -->
+  <joint name="hokuyo_joint" type="fixed">
+    <origin xyz="0.15 0 0.1" rpy="0 0 0" />
+    <parent link="chassis" />
+    <child link="hokuyo" />
+  </joint>
+  <link name='hokuyo'>
+    <pose>0 0 0 0 0 0</pose>
+    <inertial>
+      <mass value="0.1"/>
+      <origin xyz="0 0 0" rpy="0 0 0" />
+      <inertia
+          ixx="1e-6" ixy="0" ixz="0"
+          iyy="1e-6" iyz="0"
+          izz="1e-6"
+      />
+    </inertial>
+    <collision>
+      <origin xyz="0 0 0" rpy=" 0 0 0" />
+      <geometry>
+        <box size="0.1 0.1 0.1" />
+      </geometry>
+    </collision>
+    <visual>
+      <origin xyz="0 0 0" rpy=" 0 0 0" />
+      <geometry>
+        <mesh filename="package://udacity_bot/meshes/hokuyo.dae"/>
+      </geometry>
+    </visual>
+  </link>
 </robot>
